File: eagle-pcb/6502-shield/6502-shield.sch (EAGLE design)
At the start: 0 parts

Commit message: Dead end =(
Parts:
- added C1: 1uF, rcl:C-USC0805
- added C2, C5, C7: 0.01uF, rcl:C-USC0402
- added C3, C4, C6: 0.1uF, rcl:C-USC0402
- added CON1: M20-7821646-FEM-HDR, 6502-shield:M20-7821646-FEM-HDR
- added PCB1: ARDUINO_MEGA2560, E14_Arduino_revC:ARDUINO_MEGA2560
- added R1, R2, R3, R5, R7: 1K, rcl:R-US_R0603
- added R4: 1M, rcl:R-US_R0603
- added R6: 1M, 6502-shield:TRIMPOTTC33X
- added SW1: MCSLPT4644B1TR-TACT-SW, 6502-shield:MCSLPT4644B1TR-TACT-SW
- added SW2: PCM12SMTR-SPDT-RIGHT-ANG, 6502-shield:PCM12SMTR-SPDT-RIGHT-ANG
- added U1: AT28C256TSOP-28, 6502-shield:AT28C256TSOP-28
- added U13: 74HC32TSSOP-14, 6502-shield:74HC32TSSOP-14
- added U17: 74HC04TSSOP-14, 6502-shield:74HC04TSSOP-14
- added U2: W65C02S, 6502-shield:W65C02S
- added U3: AS6C62256, 6502-shield:AS6C62256
- added U4: W65C22, 6502-shield:W65C22
- added U5: MM74HC00TSSOP, 6502-shield:MM74HC00TSSOP
- added U6, U7, U8: SE555QS, 6502-shield:SE555QS
Connections:
- new net A0: U1.A0, U2.A0, U3.A0, U4.RS0
- new net A1: U1.A1, U2.A1, U3.A1, U4.RS1
- new net A10: U1.A10, U2.A10, U3.A10
- new net A11: U1.A11, U2.A11, U3.A11
- new net A12: U1.A12, U2.A12, U3.A12
- new net A13: U1.A13, U2.A13, U3.A13
- new net A14: U1.A14, U2.A14, U3.A14
- new net A15: U2.A15
- new net A2: U1.A2, U2.A2, U3.A2, U4.RS2
- new net A3: U1.A3, U2.A3, U3.A3, U4.RS3
- new net A4: U1.A4, U2.A4, U3.A4
- new net A5: U1.A5, U2.A5, U3.A5
- new net A6: U1.A6, U2.A6, U3.A6
- new net A7: U1.A7, U2.A7, U3.A7
- new net A8: U1.A8, U2.A8, U3.A8
- new net A9: U1.A9, U2.A9, U3.A9
- new net CLK: U4.PHI2, U5G$3.Y
- new net CLK_0: U5G$1.A, U6.OUT
- new net CLK_1: U5G$2.B, U7.OUT
- new net CLK_HALT: U17G$2.A
- new net CLK_SELECT: U17G$1.A, U5G$1.B, U8.OUT
- new net D0: U1.I/O0, U2.D0, U3.DQ0, U4.D0
- new net D1: U1.I/O1, U2.D1, U3.DQ1, U4.D1
- new net D2: U1.I/O2, U2.D2, U3.DQ2, U4.D2
- new net D3: U1.I/O3, U2.D3, U3.DQ3, U4.D3
- new net D4: U1.I/O4, U2.D4, U3.DQ4, U4.D4
- new net D5: U1.I/O5, U2.D5, U3.DQ5, U4.D5
- new net D6: U1.I/O6, U2.D6, U3.DQ6, U4.D6
- new net D7: U1.I/O7, U2.D7, U3.DQ7, U4.D7
- new net GND: C1.2, C2.2, C3.2, C4.2, C5.2, C6.2, C7.2, PCB1.GND, PCB1.GND., PCB1.GND.., PCB1.GND..., PCB1.GND...., SW1.T2, SW2.1, U1.GND, U13G$5.GND, U17G$7.GND, U2.VSS@1, U2.VSS@2, U2.VSS@3, U3.VSS, U4.VSS, U5G$5.GND, U6.GND, U7.GND, U8.GND, U8.THRES
- new net N$1: R2.2, R6.S
- new net N$10: U17G$1.Y, U5G$2.A
- new net N$11: U13G$1.A, U5G$1.Y
- new net N$12: U13G$1.B, U5G$2.Y
- new net N$13: U13G$1.Y, U5G$3.A
- new net N$14: U17G$2.Y, U5G$3.B
- new net N$2: C2.1, U6.CONT
- new net N$3: R1.1, R2.1, U6.DISCH
- new net N$4: R3.1, SW1.T3, U7.TRIG
- new net N$5: C5.1, U7.CONT
- new net N$6: C6.1, R4.1, U7.DISCH, U7.THRES
- new net N$7: R5.1, SW2.2, U8.TRIG
- new net N$8: R7.1, SW2.3, U8.RESET
- new net N$9: C7.1, U8.CONT
- new net PA0: U4.PA0
- new net PA1: U4.PA1
- new net PA2: U4.PA2
- new net PA3: U4.PA3
- new net PA4: U4.PA4
- new net PA5: CON1.4, U4.PA5
- new net PA6: CON1.5, U4.PA6
- new net PA7: CON1.6, U4.PA7
- new net PB0: CON1.7, U4.PB0
- new net PB1: CON1.8, U4.PB1
- new net PB2: CON1.9, U4.PB2
- new net PB3: CON1.10, U4.PB3
- new net PB4: CON1.11, U4.PB4
- new net PB5: CON1.12, U4.PB5
- new net PB6: CON1.13, U4.PB6
- new net PB7: CON1.14, U4.PB7
- new net TRIG: C1.1, R6.E, U6.THRES, U6.TRIG
- new net VCC: C3.1, C4.1, PCB1.+5V., PCB1.+5V.., PCB1.5V, R1.2, R3.2, R4.2, R5.2, R7.2, U1.VCC, U13G$5.VCC, U17G$7.VCC, U2.VDD@1, U2.VDD@2, U3.VCC, U4.VDD, U5G$5.VCC, U6.RESET, U6.VCC, U7.RESET, U7.VCC, U8.VCC
