File: eagle-pcb/6502-shield/6502-shield.sch (EAGLE design)
At the start: 38 parts

Commit message: Bunch of work on rev b. but more to do.
Parts:
- added C10, C11, C12, C13, C14, C15, C16, C17, C18, C19, C20, C21, C22, C23, C24, C25, C26, C27, C28, C8, C9: 0.1uF, rcl:C-USC0805
- added U1, U2, U3, U4, U5, U6: TCB0108-LVL-XLTRTSSOP20, 6502-shield:TCB0108-LVL-XLTRTSSOP20
- C1, C2, C3, C4, C5, C6, C7: device rcl:C-USC0402 -> rcl:C-USC0805
- R18, R2, R3, R4, R5, R6, R7, R8, R9: device rcl:R-US_R0402 -> rcl:R-US_R0603
Connections:
- new net A0_IO: PCB1.44, U2_BUFF_1.B
- new net A10_IO: PCB1.34, U1_BUFF_3.B
- new net A11_IO: PCB1.35, U1_BUFF_4.B
- new net A12_IO: PCB1.32, U1_BUFF_5.B
- new net A13_IO: PCB1.33, U1_BUFF_6.B
- new net A14_IO: PCB1.30, U1_BUFF_7.B
- new net A15_IO: PCB1.31, U1_BUFF_8.B
- new net A1_IO: PCB1.45, U2_BUFF_2.B
- new net A2_IO: PCB1.42, U2_BUFF_3.B
- new net A3_IO: PCB1.43, U2_BUFF_4.B
- new net A4_IO: PCB1.40, U2_BUFF_5.B
- new net A5_IO: PCB1.41, U2_BUFF_6.B
- new net A6_IO: PCB1.38, U2_BUFF_7.B
- new net A7_IO: PCB1.39, U2_BUFF_8.B
- new net A8_IO: PCB1.36, U1_BUFF_1.B
- new net A9_IO: PCB1.37, U1_BUFF_2.B
- new net CLK_IO: PCB1.27, U6_BUFF_5.B
- new net D0_IO: PCB1.52, U3_BUFF_1.B
- new net D1_IO: PCB1.53, U3_BUFF_2.B
- new net D2_IO: PCB1.50, U3_BUFF_3.B
- new net D3_IO: PCB1.51, U3_BUFF_4.B
- new net D4_IO: PCB1.48, U3_BUFF_5.B
- new net D5_IO: PCB1.49, U3_BUFF_6.B
- new net D6_IO: PCB1.46, U3_BUFF_7.B
- new net D7_IO: PCB1.47, U3_BUFF_8.B
- new net DMA_IO: PCB1.22, U6_BUFF_6.B
- new net EEPROM_PGM_IO: PCB1.23, U6_BUFF_2.B
- new net IRQ_COPROC: FPGA_BANK3_LEFT.PL3A, U6_BUFF_3.A
- new net IRQ_COPROC_IO: PCB1.24, U6_BUFF_3.B
- new net IRQ_IO: FPGA_BANK3_LEFT.PL3B, PIO.IRQB
- new net OE_IO: PCB1.25, U6_BUFF_1.B
- new net PA0_IO: JP2.1, U4_BUFF_8.B
- new net PA1_IO: JP2.3, U4_BUFF_7.B
- new net PA2_IO: JP2.5, U4_BUFF_6.B
- new net PA3_IO: JP2.7, U4_BUFF_5.B
- new net PA4_IO: JP2.9, U4_BUFF_4.B
- new net PA5_IO: JP2.11, U4_BUFF_3.B
- new net PA6_IO: JP2.13, U4_BUFF_2.B
- new net PA7_IO: JP2.15, U4_BUFF_1.B
- new net PB0_IO: JP2.2, U5_BUFF_8.B
- new net PB1_IO: JP2.4, U5_BUFF_7.B
- new net PB2_IO: JP2.6, U5_BUFF_6.B
- new net PB3_IO: JP2.8, U5_BUFF_5.B
- new net PB4_IO: JP2.10, U5_BUFF_4.B
- new net PB5_IO: JP2.12, U5_BUFF_3.B
- new net PB6_IO: JP2.14, U5_BUFF_2.B
- new net PB7_IO: JP2.16, U5_BUFF_1.B
- new net VCCIO: C14.1, C15.1, C16.1, C17.1, C18.1, C19.1, JP3.1, PCB1.+5V., PCB1.+5V.., PCB1.5V, U1_CORE.VCC_B, U2_CORE.VCC_B, U3_CORE.VCC_B, U4_CORE.VCC_B, U5_CORE.VCC_B, U6_CORE.VCC_B
- new net WE_IO: PCB1.29, U6_BUFF_4.B
- net A0: now also U2_BUFF_1.A; no longer PCB1.44
- net A1: now also U2_BUFF_2.A; no longer PCB1.45
- net A10: now also U1_BUFF_3.A; no longer PCB1.34
- net A11: now also U1_BUFF_4.A; no longer PCB1.35
- net A12: now also U1_BUFF_5.A; no longer PCB1.32
- net A13: now also U1_BUFF_6.A; no longer PCB1.33
- net A14: now also U1_BUFF_7.A; no longer PCB1.30
- net A15: now also U1_BUFF_8.A; no longer PCB1.31
- net A2: now also U2_BUFF_3.A; no longer PCB1.42
- net A3: now also U2_BUFF_4.A; no longer PCB1.43
- net A4: now also U2_BUFF_5.A; no longer PCB1.40
- net A5: now also U2_BUFF_6.A; no longer PCB1.41
- net A6: now also U2_BUFF_7.A; no longer PCB1.38
- net A7: now also U2_BUFF_8.A; no longer PCB1.39
- net A8: now also U1_BUFF_1.A; no longer PCB1.36
- net A9: now also U1_BUFF_2.A; no longer PCB1.37
- net CLK: now also U6_BUFF_5.A; no longer PCB1.27
- net D0: now also U3_BUFF_1.A; no longer PCB1.52
- net D1: now also U3_BUFF_2.A; no longer PCB1.53
- net D2: now also U3_BUFF_3.A; no longer PCB1.50
- net D3: now also U3_BUFF_4.A; no longer PCB1.51
- net D4: now also U3_BUFF_5.A; no longer PCB1.48
- net D5: now also U3_BUFF_6.A; no longer PCB1.49
- net D6: now also U3_BUFF_7.A; no longer PCB1.46
- net D7: now also U3_BUFF_8.A; no longer PCB1.47
- net DMA: now also U6_BUFF_6.A; no longer PCB1.22
- net EEPROM_PGM: now also U6_BUFF_2.A; no longer PCB1.23
- net GND: now also C10.2, C11.2, C12.2, C13.2, C14.2, C15.2, C16.2, C17.2, C18.2, C19.2, C20.2, C21.2, C22.2, C23.2, C24.2, C25.2, C26.2, C27.2, C28.2, C8.2, C9.2, U1_CORE.GND, U2_CORE.GND, U3_CORE.GND, U4_CORE.GND, U5_CORE.GND, U6_BUFF_7.A, U6_BUFF_8.A, U6_CORE.GND
- net IRQN: no longer PIO.IRQB
- net OE: now also U6_BUFF_1.A; no longer PCB1.25
- net PA0: now also U4_BUFF_8.A; no longer JP2.1
- net PA1: now also U4_BUFF_7.A; no longer JP2.3
- net PA2: now also U4_BUFF_6.A; no longer JP2.5
- net PA3: now also U4_BUFF_5.A; no longer JP2.7
- net PA4: now also U4_BUFF_4.A; no longer JP2.9
- net PA5: now also U4_BUFF_3.A; no longer JP2.11
- net PA6: now also U4_BUFF_2.A; no longer JP2.13
- net PA7: now also U4_BUFF_1.A; no longer JP2.15
- net PB0: now also U5_BUFF_8.A; no longer JP2.2
- net PB1: now also U5_BUFF_7.A; no longer JP2.4
- net PB2: now also U5_BUFF_6.A; no longer JP2.6
- net PB3: now also U5_BUFF_5.A; no longer JP2.8
- net PB4: now also U5_BUFF_4.A; no longer JP2.10
- net PB5: now also U5_BUFF_3.A; no longer JP2.12
- net PB6: now also U5_BUFF_2.A; no longer JP2.14
- net PB7: now also U5_BUFF_1.A; no longer JP2.16
- net TCK: now also JP1.4; no longer JP1.6
- net TDI: now also JP1.3; no longer JP1.4
- net TMS: now also JP1.6; no longer JP1.3
- net VCC: now also C10.1, C11.1, C12.1, C13.1, C20.1, C21.1, C22.1, C23.1, C24.1, C25.1, C26.1, C27.1, C28.1, C8.1, C9.1, U1_CORE.OE, U1_CORE.VCC_A, U2_CORE.OE, U2_CORE.VCC_A, U3_CORE.OE, U3_CORE.VCC_A, U4_CORE.OE, U4_CORE.VCC_A, U5_CORE.OE, U5_CORE.VCC_A, U6_CORE.OE, U6_CORE.VCC_A; no longer JP3.1
- net WE: now also U6_BUFF_4.A; no longer PCB1.29

Commit message: More routing work on the pcb, lots more left... yay =/
Connections:
- net CLK: now also U6_BUFF_2.A; no longer U6_BUFF_5.A
- net CLK_IO: now also U6_BUFF_2.B; no longer U6_BUFF_5.B
- net EEPROM_PGM: now also U6_BUFF_5.A; no longer U6_BUFF_2.A
- net EEPROM_PGM_IO: now also U6_BUFF_5.B; no longer U6_BUFF_2.B
- net IRQ_COPROC: now also U6_BUFF_4.A; no longer U6_BUFF_3.A
- net IRQ_COPROC_IO: now also U6_BUFF_4.B; no longer U6_BUFF_3.B
- net OE: now also U6_BUFF_3.A; no longer U6_BUFF_1.A
- net OE_IO: now also U6_BUFF_3.B; no longer U6_BUFF_1.B
- net PB0: now also U5_BUFF_1.A; no longer U5_BUFF_8.A
- net PB0_IO: now also U5_BUFF_1.B; no longer U5_BUFF_8.B
- net PB1: now also U5_BUFF_2.A; no longer U5_BUFF_7.A
- net PB1_IO: now also U5_BUFF_2.B; no longer U5_BUFF_7.B
- net PB2: now also U5_BUFF_3.A; no longer U5_BUFF_6.A
- net PB2_IO: now also U5_BUFF_3.B; no longer U5_BUFF_6.B
- net PB3: now also U5_BUFF_4.A; no longer U5_BUFF_5.A
- net PB3_IO: now also U5_BUFF_4.B; no longer U5_BUFF_5.B
- net PB4: now also U5_BUFF_5.A; no longer U5_BUFF_4.A
- net PB4_IO: now also U5_BUFF_5.B; no longer U5_BUFF_4.B
- net PB5: now also U5_BUFF_6.A; no longer U5_BUFF_3.A
- net PB5_IO: now also U5_BUFF_6.B; no longer U5_BUFF_3.B
- net PB6: now also U5_BUFF_7.A; no longer U5_BUFF_2.A
- net PB6_IO: now also U5_BUFF_7.B; no longer U5_BUFF_2.B
- net PB7: now also U5_BUFF_8.A; no longer U5_BUFF_1.A
- net PB7_IO: now also U5_BUFF_8.B; no longer U5_BUFF_1.B
- net WE: now also U6_BUFF_1.A; no longer U6_BUFF_4.A
- net WE_IO: now also PCB1.28, U6_BUFF_1.B; no longer PCB1.29, U6_BUFF_4.B
