File: eagle-pcb/6502-shield/6502-shield.sch (EAGLE design)
At the start: 65 parts, among them U1 TCB0108-LVL-XLTRTSSOP20, U2 TCB0108-LVL-XLTRTSSOP20, U3 TCB0108-LVL-XLTRTSSOP20, U4 TCB0108-LVL-XLTRTSSOP20, U5 TCB0108-LVL-XLTRTSSOP20, U6 TCB0108-LVL-XLTRTSSOP20

Commit message: Made some tweaks and random clean up.  Updating the images and a system block diagram.
Other:
- moved on the sheet: FPGA_BANK1_RIGHT, JP2
